File: PCB/tronzpad.kicad_pcb (KiCad board)
At the start: 2 copper layers, 13 parts, among them U1 XIAO-RP2040-DIP

Commit message: add loads of stuff to production
Parts:
- added D1: Diode, Diode_THT:D_DO-35_SOD27_P7.62mm_Horizontal, B.Cu at (119.5, 84.6)
- added D10: Diode, Diode_THT:D_DO-35_SOD27_P7.62mm_Horizontal, B.Cu at (138.5, 122.7)
- added D11: Diode, Diode_THT:D_DO-35_SOD27_P7.62mm_Horizontal, B.Cu at (157.6, 122.7)
- added D12: Diode, Diode_THT:D_DO-35_SOD27_P7.62mm_Horizontal, B.Cu at (176.6, 122.7)
- added D13: LED_SK6812MINI, ScottoKeebs_Components:LED_SK6812MINI, B.Cu at (129.0, 86.5)
- added D14: LED_SK6812MINI, ScottoKeebs_Components:LED_SK6812MINI, B.Cu at (148.1, 86.5)
- added D15: LED_SK6812MINI, ScottoKeebs_Components:LED_SK6812MINI, B.Cu at (167.2, 86.5)
- added D16: LED_SK6812MINI, ScottoKeebs_Components:LED_SK6812MINI, B.Cu at (148.1, 105.6)
- added D17: LED_SK6812MINI, ScottoKeebs_Components:LED_SK6812MINI, B.Cu at (129.0, 105.6)
- added D18: LED_SK6812MINI, ScottoKeebs_Components:LED_SK6812MINI, B.Cu at (110.0, 105.6)
- added D19: LED_SK6812MINI, ScottoKeebs_Components:LED_SK6812MINI, B.Cu at (110.0, 124.6)
- added D2: Diode, Diode_THT:D_DO-35_SOD27_P7.62mm_Horizontal, B.Cu at (138.5, 84.6)
- added D20: LED_SK6812MINI, ScottoKeebs_Components:LED_SK6812MINI, B.Cu at (129.0, 124.6)
- added D21: LED_SK6812MINI, ScottoKeebs_Components:LED_SK6812MINI, B.Cu at (167.1, 105.6)
- added D22: LED_SK6812MINI, ScottoKeebs_Components:LED_SK6812MINI, B.Cu at (148.1, 124.6)
- added D23: LED_SK6812MINI, ScottoKeebs_Components:LED_SK6812MINI, B.Cu at (167.1, 124.6)
- added D24: LED_SK6812MINI, ScottoKeebs_Components:LED_SK6812MINI, B.Cu at (174.1, 68.3)
- added D25: LED_SK6812MINI, ScottoKeebs_Components:LED_SK6812MINI, B.Cu at (110.0, 86.5)
- added D26: LED_SK6812MINI, ScottoKeebs_Components:LED_SK6812MINI, B.Cu at (177.5, 68.3)
- added D27: LED_SK6812MINI, ScottoKeebs_Components:LED_SK6812MINI, B.Cu at (181.0, 68.3)
- added D3: Diode, Diode_THT:D_DO-35_SOD27_P7.62mm_Horizontal, B.Cu at (157.6, 84.6)
- added D4: Diode, Diode_THT:D_DO-35_SOD27_P7.62mm_Horizontal, B.Cu at (176.6, 84.6)
- added D5: Diode, Diode_THT:D_DO-35_SOD27_P7.62mm_Horizontal, B.Cu at (119.5, 103.7)
- added D6: Diode, Diode_THT:D_DO-35_SOD27_P7.62mm_Horizontal, B.Cu at (138.5, 103.7)
- added D7: Diode, Diode_THT:D_DO-35_SOD27_P7.62mm_Horizontal, B.Cu at (157.6, 103.7)
- added D8: Diode, Diode_THT:D_DO-35_SOD27_P7.62mm_Horizontal, B.Cu at (176.1, 103.5)
- added D9: Diode, Diode_THT:D_DO-35_SOD27_P7.62mm_Horizontal, B.Cu at (119.5, 122.7)
- added G***: LOGO, LOGO, F.Cu at (187.8, 119.8)
- added G***: LOGO, LOGO, F.Cu at (187.8, 103.2)
- added G***: LOGO, LOGO, F.Cu at (122.5, 68.5)
- added G***: LOGO, LOGO, F.Cu at (191.9, 125.4)
- added G***: LOGO, LOGO, F.Cu at (131.2, 132.8)
- added G***: LOGO, LOGO, F.Cu at (183.6, 125.3)
- added G***: LOGO, LOGO, F.Cu at (138.6, 91.2)
- added G***: LOGO, LOGO, F.Cu at (117.6, 98.7)
- added G***: LOGO, LOGO, F.Cu at (188.0, 99.1)
- added G***: LOGO, LOGO, F.Cu at (187.8, 115.0)
- added H1: Mounting_Hole, MountingHole:MountingHole_3.2mm_M3_DIN965, F.Cu at (103.6, 68.6)
- added H2: Mounting_Hole, MountingHole:MountingHole_3.2mm_M3_DIN965, F.Cu at (194.4, 68.6)
- added H3: Mounting_Hole, MountingHole:MountingHole_3.2mm_M3_DIN965, F.Cu at (103.6, 132.6)
- added H4: Mounting_Hole, MountingHole:MountingHole_3.2mm_M3_DIN965, F.Cu at (194.4, 132.6)
- added SW1: RotaryEncoder_Switch_MP, Rotary_Encoder:RotaryEncoder_Alps_EC11E-Switch_Vertical_H20mm, F.Cu at (186.0, 88.9)
- moved S10 114.8 mm to (131.5, 114.8)
- moved S9 108.3 mm to (112.5, 114.8)
- moved S5 92.7 mm to (112.5, 95.7)
- moved S11 91.0 mm to (150.6, 114.8)
- moved S1 77.2 mm to (112.5, 76.7)
- moved S7 75.7 mm to (150.6, 95.7)
- moved S6 71.9 mm to (131.5, 95.7)
- moved S12 67.7 mm to (169.6, 114.8)
- moved S2 56.7 mm to (131.5, 76.7)
- moved S8 52.2 mm to (169.6, 95.7)
- moved U1 42.5 mm to (188.1, 101.2), turned to -90 degrees
- moved S3 40.8 mm to (150.6, 76.7)
- moved S4 36.7 mm to (169.6, 76.7)
Connections:
- S1 pad 1: COLUMN 1 -> Net-(D1-A)
- S1 pad 2: Net-(D1-A) -> COLUMN 1
- S10 pad 1: COLUMN 2 -> Net-(D10-A)
- S10 pad 2: Net-(D10-A) -> COLUMN 2
- S11 pad 1: COLUMN 3 -> Net-(D11-A)
- S11 pad 2: Net-(D11-A) -> COLUMN 3
- S12 pad 1: COLUMN 4 -> Net-(D12-A)
- S12 pad 2: Net-(D12-A) -> COLUMN 4
- S2 pad 1: COLUMN 2 -> Net-(D2-A)
- S2 pad 2: Net-(D2-A) -> COLUMN 2
- S3 pad 1: COLUMN 3 -> Net-(D3-A)
- S3 pad 2: Net-(D3-A) -> COLUMN 3
- S4 pad 1: COLUMN 4 -> Net-(D4-A)
- S4 pad 2: Net-(D4-A) -> COLUMN 4
- S5 pad 1: COLUMN 1 -> Net-(D5-A)
- S5 pad 2: Net-(D5-A) -> COLUMN 1
- S6 pad 1: COLUMN 2 -> Net-(D6-A)
- S6 pad 2: Net-(D6-A) -> COLUMN 2
- S7 pad 1: COLUMN 3 -> Net-(D7-A)
- S7 pad 2: Net-(D7-A) -> COLUMN 3
- S8 pad 1: COLUMN 4 -> Net-(D8-A)
- S8 pad 2: Net-(D8-A) -> COLUMN 4
- S9 pad 1: COLUMN 1 -> Net-(D9-A)
- S9 pad 2: Net-(D9-A) -> COLUMN 1
- U1 pad 12: unconnected-(U1-3V3-Pad12) -> 3.3V
- U1 pad 13: unconnected-(U1-GND-Pad13) -> GND
- U1 pad 14: unconnected-(U1-VBUS-Pad14) -> VBUS
- U1 pad 5: unconnected-(U1-GPIO6/SDA-Pad5) -> ROTARY 1
- U1 pad 6: unconnected-(U1-GPIO7/SCL-Pad6) -> ROTARY 2
- U1 pad 7: unconnected-(U1-GPIO0/TX-Pad7) -> ROTARY 3
- U1 pad 8: unconnected-(U1-GPIO1/RX-Pad8) -> RGB_LED
Routing:
- net COLUMN 1: track 0.00 -> 173.3 mm
- net COLUMN 2: track 0.00 -> 169.8 mm
- net COLUMN 3: track 0.00 -> 124.6 mm
- net COLUMN 4: track 0.00 -> 103.0 mm
- net RGB_LED: track 0.00 -> 90.1 mm, vias 0 -> 2
- net ROW 1: track 0.00 -> 87.3 mm, vias 0 -> 2
- net ROW 3: track 0.00 -> 79.3 mm
- net Net-(D23-DOUT): track 0.00 -> 77.0 mm, vias 0 -> 6
- net GND: track 0.00 -> 70.8 mm, vias 0 -> 24
- net ROW 2: track 0.00 -> 70.2 mm
- net VBUS: track 0.00 -> 54.1 mm, vias 0 -> 14
- net Net-(D24-DOUT): track 0.00 -> 26.6 mm, vias 0 -> 2
- net ROTARY 1: track 0.00 -> 26.5 mm
- net Net-(D15-DOUT): track 0.00 -> 25.4 mm
- net Net-(D18-DOUT): track 0.00 -> 20.7 mm
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- added copper zone on F.Cu, net GND
- added copper zone on B.Cu, net VBUS
Other:
- board outline added: 99.8 x 73 mm
- board text added: "EC11"
- board text added: "VBUS"
