File: PCB/tronzpad.kicad_sch (KiCad schematic)
At the start: 42 parts, among them SW1 RotaryEncoder_Switch_MP, U1 XIAO-RP2040-DIP

Commit message: add loads of stuff to production
Parts:
- added D24, D26, D27: LED_SK6812MINI, ScottoKeebs_Components:LED_SK6812MINI, symbol ScottoKeebs:LED_SK6812MINI
Connections:
- net COLUMN 4 is gone; now on net COLUMN 3: S12.2, S4.2, S8.2, U1.4 (GPIO29/ADC3/A3)
- net ROW 3 is gone; now on net ROW 2: D10.1 (K), D11.1 (K), D12.1 (K), D9.1 (K), U1.9 (GPIO2/SCK)
- net COLUMN 1: now also S10.2, S2.2, S6.2, U1.2 (GPIO27/ADC1/A1); no longer S1.2, S5.2, S9.2, U1.1 (GPIO26/ADC0/A0)
- net COLUMN 2: now also S11.2, S3.2, S7.2, U1.3 (GPIO28/ADC2/A2); no longer S10.2, S2.2, S6.2, U1.2 (GPIO27/ADC1/A1)
- net COLUMN 3: no longer S11.2, S3.2, S7.2, U1.3 (GPIO28/ADC2/A2)
- net GND: now also D24.3 (VSS), D26.3 (VSS), D27.3 (VSS)
- net ROW 1: now also D5.1 (K), D6.1 (K), D7.1 (K), D8.1 (K), U1.10 (GPIO4/MISO); no longer D1.1 (K), D2.1 (K), D3.1 (K), D4.1 (K), U1.11 (GPIO3/MOSI)
- net ROW 2: no longer D5.1 (K), D6.1 (K), D7.1 (K), D8.1 (K), U1.10 (GPIO4/MISO)
- net VBUS: now also D24.1 (VDD), D26.1 (VDD), D27.1 (VDD)
- net at D23.2 (DOUT): now also D24.4 (DIN)
- new net: D26.2 (DOUT), D27.4 (DIN)
- new net: D24.2 (DOUT), D26.4 (DIN)
- new net COLUMN 0: S1.2, S5.2, S9.2, U1.1 (GPIO26/ADC0/A0)
- new net ROW 0: D1.1 (K), D2.1 (K), D3.1 (K), D4.1 (K), U1.11 (GPIO3/MOSI)
Other:
- note added: "MOUNTING HOLES"
- note added: "STATUS LED"
- moved on the sheet: H1, H2, H3, H4, U1
